File: bbb_indexer_r1/bbb_indexer_r1.kicad_pcb (KiCad board)
At the start: 2 copper layers, 54.6 x 86.4 mm, 39 parts, among them J1 SS-60000-008-stepdir, J2 SS-60000-008-stepdir, J3 SS-60000-008-stepdir, J4 SS-60000-008-stepdir, J5 SS-60000-008-stepdir, J6 SS-60000-008-stepdir, J7 Conn_01x02, J8 Conn_02x05_Odd_Even, P8 BeagleBone_Black_Header_P8, P9 BeagleBone_Black_Header_P9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

Commit message: bbb_indexer_r1-rc5 I think
Signed-off-by: John McMaster <johndmcmaster@gmail.com>
Other:
- board text added: "BBB INDEXER R1 JOHN MCMASTER 2018"
Changed lines of the file:
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@@
     (links 148)
     (no_connects 0)
-    (area 105.098651 42.2086 175.901548 130.137305)
+    (area 114.463829 42.696129 169.076371 129.058671)
     (thickness 1.6)
-    (drawings 11)
+    (drawings 12)
     (tracks 2040)
     (zones 0)
@@
     (mod_text_size 1 1)
     (mod_text_width 0.15)
-    (pad_size 1.7272 1.7272)
-    (pad_drill 1.016)
+    (pad_size 3.175 3.175)
+    (pad_drill 3.175)
     (pad_to_mask_clearance 0)
     (aux_axis_origin 0 0)
@@
     )
   )
+  (gr_text "BBB INDEXER R1\nJOHN MCMASTER\n2018" (at 121.666 51.816) (layer F.SilkS)
+    (effects (font (size 1.016 1.016) (thickness 0.1905)))
+  )
   (gr_line (start 127.1651 129.0574) (end 156.3751 129.0574) (layer Edge.Cuts) (width 0.00254))
   (gr_line (start 135.4201 64.2874) (end 135.4201 42.6974) (layer Edge.Cuts) (width 0.00254))
@@
   (segment (start 121.158 87.122) (end 121.158 87.606933) (width 0.1524) (layer F.Cu) (net 110))
   (via (at 121.158 87.122) (size 0.6858) (drill 0.3302) (layers F.Cu B.Cu) (net 110))
-  (segment (start 131.737101 95.238161) (end 132.087575 94.887687) (width 0.1524) (layer F.Cu) (net 111))
-  (segment (start 131.737101 99.997285) (end 131.737101 95.238161) (width 0.1524) (layer F.Cu) (net 111))
-  (segment (start 132.02922 100.289403) (end 131.737101 99.997285) (width 0.1524) (layer F.Cu) (net 111))
-  (segment (start 132.02922 102.910598) (end 132.02922 100.289403) (width 0.1524) (layer F.Cu) (net 111))
-  (segment (start 131.737101 103.202717) (end 132.02922 102.910598) (width 0.1524) (layer F.Cu) (net 111))
-  (segment (start 131.737101 105.321101) (end 131.737101 103.202717) (width 0.1524) (layer F.Cu) (net 111))
-  (segment (start 132.08 105.664) (end 131.737101 105.321101) (width 0.1524) (layer F.Cu) (net 111))
   (segment (start 132.087575 94.887687) (end 132.087575 93.92922) (width 0.1524) (layer F.Cu) (net 111))
   (segment (start 132.087575 93.92922) (end 131.744676 93.586321) (width 0.1524) (layer F.Cu) (net 111))
+  (segment (start 131.737101 95.238161) (end 132.087575 94.887687) (width 0.1524) (layer F.Cu) (net 111))
+  (segment (start 132.08 105.664) (end 131.737101 105.321101) (width 0.1524) (layer F.Cu) (net 111))
+  (segment (start 131.737101 105.321101) (end 131.737101 103.202717) (width 0.1524) (layer F.Cu) (net 111))
+  (segment (start 131.737101 103.202717) (end 132.02922 102.910598) (width 0.1524) (layer F.Cu) (net 111))
+  (segment (start 132.02922 102.910598) (end 132.02922 100.289403) (width 0.1524) (layer F.Cu) (net 111))
+  (segment (start 132.02922 100.289403) (end 131.737101 99.997285) (width 0.1524) (layer F.Cu) (net 111))
+  (segment (start 131.737101 99.997285) (end 131.737101 95.238161) (width 0.1524) (layer F.Cu) (net 111))
+  (segment (start 143.4592 109.1154) (end 143.4592 109.5654) (width 0.1524) (layer B.Cu) (net 111))
+  (segment (start 140.5158 106.172) (end 143.4592 109.1154) (width 0.1524) (layer B.Cu) (net 111))
+  (segment (start 132.588 106.172) (end 140.5158 106.172) (width 0.1524) (layer B.Cu) (net 111))
+  (segment (start 132.08 105.664) (end 132.588 106.172) (width 0.1524) (layer B.Cu) (net 111))
+  (via (at 132.08 105.664) (size 0.6858) (drill 0.3302) (layers F.Cu B.Cu) (net 111))
   (segment (start 125.274267 92.8624) (end 125.731488 93.319622) (width 0.1524) (layer B.Cu) (net 111))
   (segment (start 118.9101 92.8624) (end 125.274267 92.8624) (width 0.1524) (layer B.Cu) (net 111))
@@
   (segment (start 131.303813 93.586321) (end 131.744676 93.586321) (width 0.1524) (layer B.Cu) (net 111))
   (via (at 131.744676 93.586321) (size 0.6858) (drill 0.3302) (layers F.Cu B.Cu) (net 111))
-  (segment (start 132.588 106.172) (end 140.5158 106.172) (width 0.1524) (layer B.Cu) (net 111))
-  (segment (start 140.5158 106.172) (end 143.4592 109.1154) (width 0.1524) (layer B.Cu) (net 111))
-  (segment (start 143.4592 109.1154) (end 143.4592 109.5654) (width 0.1524) (layer B.Cu) (net 111))
-  (segment (start 132.08 105.664) (end 132.588 106.172) (width 0.1524) (layer B.Cu) (net 111))
-  (via (at 132.08 105.664) (size 0.6858) (drill 0.3302) (layers F.Cu B.Cu) (net 111))
   (segment (start 131.352716 95.261657) (end 131.352716 94.776724) (width 0.1524) (layer F.Cu) (net 112))
   (segment (start 131.352716 100.043966) (end 131.352716 95.261657) (width 0.1524) (layer F.Cu) (net 112))
-  (segment (start 131.724409 102.784342) (end 131.724409 100.415659) (width 0.1524) (layer F.Cu) (net 112))
-  (segment (start 131.318 103.190751) (end 131.724409 102.784342) (width 0.1524) (layer F.Cu) (net 112))
-  (segment (start 131.318 106.426) (end 131.318 103.190751) (width 0.1524) (layer F.Cu) (net 112))
   (segment (start 131.724409 100.415659) (end 131.352716 100.043966) (width 0.1524) (layer F.Cu) (net 112))
+  (segment (start 131.318 106.426) (end 131.318 103.190751) (width 0.1524) (layer F.Cu) (net 112))
+  (segment (start 131.318 103.190751) (end 131.724409 102.784342) (width 0.1524) (layer F.Cu) (net 112))
+  (segment (start 131.724409 102.784342) (end 131.724409 100.415659) (width 0.1524) (layer F.Cu) (net 112))
+  (via (at 131.318 106.426) (size 0.6858) (drill 0.3302) (layers F.Cu B.Cu) (net 112))
+  (segment (start 131.318 106.426) (end 131.660899 106.768899) (width 0.1524) (layer B.Cu) (net 112))
+  (segment (start 131.660899 106.768899) (end 137.302699 106.768899) (width 0.1524) (layer B.Cu) (net 112))
+  (segment (start 137.302699 106.768899) (end 139.6492 109.1154) (width 0.1524) (layer B.Cu) (net 112))
   (segment (start 116.3701 95.4024) (end 117.513088 96.545388) (width 0.1524) (layer B.Cu) (net 112))
   (segment (start 130.867783 94.776724) (end 131.352716 94.776724) (width 0.1524) (layer B.Cu) (net 112))
@@
   (via (at 131.352716 94.776724) (size 0.6858) (drill 0.3302) (layers F.Cu B.Cu) (net 112))
   (segment (start 139.6492 109.1154) (end 139.6492 109.5654) (width 0.1524) (layer B.Cu) (net 112))
-  (segment (start 137.302699 106.768899) (end 139.6492 109.1154) (width 0.1524) (layer B.Cu) (net 112))
-  (segment (start 131.660899 106.768899) (end 137.302699 106.768899) (width 0.1524) (layer B.Cu) (net 112))
-  (segment (start 131.318 106.426) (end 131.660899 106.768899) (width 0.1524) (layer B.Cu) (net 112))
-  (via (at 131.318 106.426) (size 0.6858) (drill 0.3302) (layers F.Cu B.Cu) (net 112))
   (segment (start 134.264433 83.413567) (end 135.4658 82.2122) (width 0.1524) (layer B.Cu) (net 115))
   (segment (start 132.725633 83.413567) (end 134.264433 83.413567) (width 0.1524) (layer B.Cu) (net 115))
